Commit message: add project lesson changes

File: src/my_robot/urdf/my_robot.xacro (robot description, xacro)
@@ -1,3 +1,4 @@
 <robot name="my_robot" xmlns:xacro="http://www.ros.org/wiki/xacro">
+    <xacro:include filename="$(find my_robot)/urdf/my_robot.gazebo"/>
     <link name="robot_footprint"></link>
     <joint name="robot_footprint_joint" type="fixed">
@@ -118,3 +119,59 @@
         <dynamics damping="1.0" friction="1.0"/>
     </joint>
+    <link name="camera">
+        <pose>0 0 0 0 0 0</pose>
+        <inertial>
+            <mass value="0.1"/>
+            <origin xyz="0 0 0" rpy="0 0 0"/>
+            <inertia
+                ixx="1e-6" ixy="0" ixz="0"
+                iyy="1e-6" iyz="0"
+                izz="1e-6"
+            />
+        </inertial>
+        <visual>
+            <geometry>
+                <box size=" 0.05 0.05 0.05"/>
+            </geometry>
+        </visual>
+        <collision>
+            <geometry>
+                <box size=" 0.05 0.05 0.05"/>
+            </geometry>
+        </collision>
+    </link>
+    <joint type="fixed" name="camera_joint">
+        <origin xyz="0.2 0 0" rpy="0 0 0"/>
+        <child link="camera"/>
+        <parent link="chassis"/>
+        <axis xyz="0 1 0" rpy="0 0 0"/>
+    </joint>
+    <link name="hokuyo">
+        <pose>0 0 0 0 0 0</pose>
+        <inertial>
+            <mass value="1e-5"/>
+            <origin xyz="0 0 0" rpy="0 0 0"/>
+            <inertia
+                ixx="1e-6" ixy="0" ixz="0"
+                iyy="1e-6" iyz="0"
+                izz="1e-6"
+            />
+        </inertial>
+        <visual>
+            <geometry>
+                <mesh filename="package://my_robot/meshes/hokuyo.dae"/>
+            </geometry>
+        </visual>
+        <collision>
+            <geometry>
+                <box size="0.1 0.1 0.1"/>
+            </geometry>
+        </collision>
+    </link>
+    <joint type="fixed" name="hokuyo_joint">
+        <origin xyz="0.15 0 0.1" rpy="0 0 0"/>
+        <child link="hokuyo"/>
+        <parent link="chassis"/>
+        <axis xyz="0 1 0" rpy="0 0 0"/>
+    </joint>
 </robot>

Commit message: build new_robot

File: src/my_robot/urdf/my_robot.xacro (robot description, xacro)
@@ -1,3 +1,3 @@
-<robot name="my_robot" xmlns:xacro="http://www.ros.org/wiki/xacro">
+<robot name="new_robot" xmlns:xacro="http://www.ros.org/wiki/xacro">
     <xacro:include filename="$(find my_robot)/urdf/my_robot.gazebo"/>
     <link name="robot_footprint"></link>
@@ -13,7 +13,7 @@
             <origin xyz="0.0 0 0" rpy=" 0 0 0"/>
             <inertia
-                ixx="0.1" ixy="0" ixz="0"
-                iyy="0.1" iyz="0"
-                izz="0.1"
+                ixx="0.2" ixy="0" ixz="0"
+                iyy="0.2" iyz="0"
+                izz="0.3"
             />
         </inertial>
@@ -21,5 +21,5 @@
             <origin xyz="0 0 0" rpy=" 0 0 0"/>
             <geometry>
-            <box size=".4 .2 .1"/>
+                <box size=".4 .2 .1"/>
             </geometry>
         </collision>
@@ -27,5 +27,5 @@
             <origin xyz="0 0 0" rpy=" 0 0 0"/>
             <geometry>
-            <box size=".4 .2 .1"/>
+                <box size=".4 .2 .1"/>
             </geometry>
         </visual>
@@ -130,10 +130,10 @@
             />
         </inertial>
-        <visual>
+        <visual name="camera_visual">
             <geometry>
                 <box size=" 0.05 0.05 0.05"/>
             </geometry>
         </visual>
-        <collision>
+        <collision name="camera_collision">
             <geometry>
                 <box size=" 0.05 0.05 0.05"/>
@@ -158,10 +158,10 @@
             />
         </inertial>
-        <visual>
+        <visual name="hokuyo_visual">
             <geometry>
                 <mesh filename="package://my_robot/meshes/hokuyo.dae"/>
             </geometry>
         </visual>
-        <collision>
+        <collision name="hokuyo_collision">
             <geometry>
                 <box size="0.1 0.1 0.1"/>
